File: c64_psu.kicad_sch (KiCad schematic)
At the start: 39 parts, among them J1 230VAC, J2 230VAC, J5 5VDC, J6 GND, J7 12VDC, J8 GND, Q1 BT145, Q2 BT145, U1 LM2596S-ADJ, U2 LM2596S-ADJ

Commit message: v2.0: Replace LM2596 with SMD type
Parts:
- U1, U2: footprint Package_TO_SOT_THT:TO-220-5_P3.4x3.7mm_StaggerOdd_Lead3.8mm_Vertical -> c64_psu:TO-263-5_TabPin3
Changed lines of the file:
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@@
 	(title_block
 		(title "C64 and 1541 PSU")
-		(date "2025-01-11")
-		(rev "1.0")
+		(date "2025-01-23")
+		(rev "2.0")
 	)
 	(junction
@@
 	(wire
 		(pts
-			(xy 43.18 69.85) (xy 69.85 69.85)
-		)
-		(stroke
-			(width 0)
-			(type default)
-		)
-	)
-	(wire
-		(pts
 			(xy 180.34 45.72) (xy 189.23 45.72)
 		)
@@
 	(wire
 		(pts
+			(xy 43.18 69.85) (xy 69.85 69.85)
+		)
+		(stroke
+			(width 0)
+			(type default)
+		)
+	)
+	(wire
+		(pts
 			(xy 173.99 143.51) (xy 173.99 144.78)
 		)
@@
 			)
 		)
-		(property "Footprint" "Package_TO_SOT_THT:TO-220-5_P3.4x3.7mm_StaggerOdd_Lead3.8mm_Vertical"
+		(property "Footprint" "c64_psu:TO-263-5_TabPin3"
 			(at 168.91 83.82 0)
 			(effects
@@
 			)
 		)
-		(property "Footprint" "Package_TO_SOT_THT:TO-220-5_P3.4x3.7mm_StaggerOdd_Lead3.8mm_Vertical"
+		(property "Footprint" "c64_psu:TO-263-5_TabPin3"
 			(at 168.91 54.61 0)
 			(effects
